File: Songbird/schematics/SBV0.3.sch (EAGLE design)
At the start: 49 parts, among them IC1 TLC2272344P, J1 AVR_SPI_PRG_6NS, U1 USD-SOCKETNEW, U2 ARDUINO_R3_SHIELDNOLABELS, U5 TLC2272344P

Commit message: Deleted uncessacary files, various updates / tweaks to model test utility
Parts:
- removed BATT: BATTERY-16MMSMD, byb:BATTERY-16MMSMD
- removed D3: (no value), SparkFun-DiscreteSemi:DIODE1N4148
- removed J10, J11, J12, J4, J5, J6, J7, J8, J9: (no value), SparkFun-Connectors:M10SILK_FEMALE_PTH
- removed J14: (no value), SparkFun-Connectors:M03PTH
- removed SJ1, SJ2: SOLDERJUMPERNC, SparkFun-Passives:SOLDERJUMPERNC
- added 3.3V, 5V, D7: SOLDERJUMPERTRACE, SparkFun:SOLDERJUMPERTRACE
- added BATT1: BATTERY-16MMSMD, byb:BATTERY-16MMSMD
- added C10, C5, C8, C9: 10uf, 1MaxBYB:M2-CAP
- added CARD, REC: (no value), SparkFun-LED:LED5MM
- added IC2: DS1307, 1MaxBYB:DS1307
- added JP2: M01SMD-4.5X1.5, 1MaxBYB:M01SMD-4.5X1.5
- added Q2: 32.768kHz, 1MaxBYB:CRYSTALTC26H
- added R11: 300, resistor:R-EU_0309/V
- added R13, R14: 4.7k, resistor:R-EU_0309/V
- added R7: 10k, resistor:R-EU_0309/V
- added S1: (no value), 1MaxBYB:TAC_SWITCHPTH
- R1, R10, R12, R16, R2, R3, R4, R5, R6, R8, R9: device 1MaxBYB:M2-RES -> resistor:R-EU_0309/V
Connections:
- removed net D2: U2.D2
- new net ASD: D7.1, IC1A.OUT, R12.1, TP8.TP
- new net GND-D: BATT1.-, C3.2, C7.2, C9.1, CARD.C, IC2.GND, JP2.1, R10.2, R7.2, REC.C, U1.GND, U1.SHIELD@1, U1.SHIELD@2, U1.SHIELD@3, U1.SHIELD@4, U2.GND@2
- new net N$13: CARD.A, U2.D13
- new net N$15: BATT1.+, IC2.VBAT
- new net PREA1: C4.2, IC1B.+IN, R6.2, R8.1
- new net SQW: IC2.SQW/OUT, U2.D2
- net 3.3V: now also 3.3V.1, 3.3V.2, C10.1, S1.3, S1.4; no longer D3.C
- net 5V: now also 5V.1, 5V.2, C5.1, C8.2, C9.2, DIVIDER.1, IC1A.V+, IC2.VCC, R13.2, R14.2; no longer IC1A.V-, J1.2
- net A1: now also IC1B.OUT, R11.2; no longer C4.2, R6.2, R8.1
- net A4: no longer SJ1.2
- net A5: no longer SJ2.2
- net D7: now also D7.2; no longer IC1A.OUT, R12.1, TP8.TP
- net GND: now also C10.2, C5.2, C8.1, IC1A.V-; no longer BATT.-, C3.2, C7.2, IC1A.V+, J1.6, R10.2, U1.GND, U1.SHIELD@1, U1.SHIELD@2, U1.SHIELD@3, U1.SHIELD@4, U2.GND@2
- net N$10: now also IC2.X2, Q2.1; no longer IC1B.OUT, J14.1
- net N$12: now also R7.1, S1.1, S1.2, U2.D12; no longer DIVIDER.1
- net N$2: now also REC.A, U2.*D11; no longer BATT.+, D3.A
- net N$8: now also IC2.X1, Q2.2; no longer IC1B.+IN, J14.3
- net N$9: now also R11.1; no longer J14.2
- net RES: no longer J1.5
- net SCL: now also IC2.SCL, R14.1; no longer SJ2.1
- net SDA: now also IC2.SDA, R13.1; no longer SJ1.1
Other:
- note added: "(Y) A/Digital Ground Bridge"
- note added: "FERRITE CHIP 3 OHM 700MA 0603 Digi-Key Part Number 445-8676-1-ND"
- note added: "I2C Address = 0x68"
- note added: "Real Time Clock and Breadboard"
- note removed: "extra Opamp"
- moved on the sheet: C1, C3, C7, IC1B, POWER, U1
